File: electronics_design/SmartLampSE.kicad_pcb (KiCad board)
At the start: 2 copper layers, 60 x 60 mm, 14 parts, among them J1 Screw_Terminal_01x02, M1 PIC16F886-IP, U1 L7805, Y1 Crystal

Commit message: Add visual polarity indicators to board supply
Routing:
- net GND: track 137.6 -> 139.1 mm
Other:
- board text added: "+"
- board text added: "-"
Changed lines of the file:
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@@
   (gr_circle (center 166 129) (end 166 133)
     (stroke (width 0.2) (type solid)) (fill none) (layer "B.Cu"))
-  (gr_rect (start 121 85) (end 161 75)
+  (gr_rect (start 121 75) (end 161 85)
     (stroke (width 0.2) (type default)) (fill none) (layer "F.SilkS"))
   (gr_circle (center 166 79) (end 168 79)
@@
   (gr_rect (start 111 74) (end 171 134)
     (stroke (width 0.2) (type solid)) (fill none) (layer "Edge.Cuts"))
+  (gr_text "+" (at 119.84 122.52) (layer "B.Cu")
+    (effects (font (size 4 4) (thickness 1) bold) (justify left bottom mirror))
+  )
   (gr_text "GND(B)" (at 164.49 112.61) (layer "B.Cu")
     (effects (font (size 1.2 1.2) (thickness 0.25) bold) (justify left bottom mirror))
@@
     (effects (font (size 1.2 1.2) (thickness 0.3) bold) (justify left bottom mirror))
   )
+  (gr_text "-" (at 119.08 103.02 90) (layer "B.Cu")
+    (effects (font (size 4 4) (thickness 1) bold) (justify left bottom mirror))
+  )
   (gr_text "PIN1" (at 134.95 86.69) (layer "B.Cu")
     (effects (font (size 1.6 1.6) (thickness 0.4) bold) (justify left bottom mirror))
@@
   (segment (start 114.066223 95.167553) (end 115.46867 96.57) (width 0.8) (layer "B.Cu") (net 2))
   (segment (start 124.87 98.81) (end 130.27 98.81) (width 0.8) (layer "B.Cu") (net 2))
+  (segment (start 120.81 109.254416) (end 119.444416 110.62) (width 0.8) (layer "B.Cu") (net 2))
   (segment (start 142.88 111.32) (end 144.62 111.32) (width 0.8) (layer "B.Cu") (net 2))
+  (segment (start 121.9501 100.65) (end 120.81 101.7901) (width 0.8) (layer "B.Cu") (net 2))
   (segment (start 136.435844 106.24) (end 137 106.24) (width 0.8) (layer "B.Cu") (net 2))
   (segment (start 131.07 98.81) (end 134.8 102.54) (width 0.8) (layer "B.Cu") (net 2))
+  (segment (start 123.03 100.65) (end 121.9501 100.65) (width 0.8) (layer "B.Cu") (net 2))
   (segment (start 130.27 121.81) (end 129.47 121.81) (width 0.8) (layer "B.Cu") (net 2))
   (segment (start 138.335 75.925) (end 133.774516 75.925) (width 0.8) (layer "B.Cu") (net 2))
@@
   (segment (start 134.8 104.604156) (end 136.435844 106.24) (width 0.8) (layer "B.Cu") (net 2))
   (segment (start 118.679516 91.02) (end 116.100995 91.02) (width 0.8) (layer "B.Cu") (net 2))
-  (segment (start 121.9501 100.65) (end 123.03 100.65) (width 0.8) (layer "B.Cu") (net 2))
   (segment (start 116.465 96.57) (end 118.95 96.57) (width 0.8) (layer "B.Cu") (net 2))
-  (segment (start 116.91 105.6901) (end 121.9501 100.65) (width 0.8) (layer "B.Cu") (net 2))
   (segment (start 124.13 100.65) (end 123.03 100.65) (width 0.8) (layer "B.Cu") (net 2))
   (segment (start 118.95 96.57) (end 123.03 100.65) (width 0.8) (layer "B.Cu") (net 2))
@@
   (segment (start 141.03 78.62) (end 138.335 75.925) (width 0.8) (layer "B.Cu") (net 2))
   (segment (start 137.8 106.24) (end 142.88 111.32) (width 0.8) (layer "B.Cu") (net 2))
-  (segment (start 116.91 110.62) (end 116.91 105.6901) (width 0.8) (layer "B.Cu") (net 2))
   (segment (start 141.03 79.975) (end 141.03 78.62) (width 0.8) (layer "B.Cu") (net 2))
   (segment (start 149.024311 107.975689) (end 145.68 111.32) (width 0.8) (layer "B.Cu") (net 2))
   (segment (start 123.03 100.65) (end 124.87 98.81) (width 0.8) (layer "B.Cu") (net 2))
+  (segment (start 120.81 101.7901) (end 120.81 109.254416) (width 0.8) (layer "B.Cu") (net 2))
   (segment (start 123.03 95.33) (end 123.02 95.32) (width 0.8) (layer "B.Cu") (net 2))
   (segment (start 114.066223 93.054772) (end 114.066223 95.167553) (width 0.8) (layer "B.Cu") (net 2))
@@
   (segment (start 115.46867 96.57) (end 116.465 96.57) (width 0.8) (layer "B.Cu") (net 2))
   (segment (start 134.8 102.54) (end 134.8 104.604156) (width 0.8) (layer "B.Cu") (net 2))
+  (segment (start 119.444416 110.62) (end 116.91 110.62) (width 0.8) (layer "B.Cu") (net 2))
   (segment (start 156 111.92) (end 156 110.427432) (width 0.8) (layer "B.Cu") (net 2))
   (segment (start 137 106.24) (end 137.8 106.24) (width 0.8) (layer "B.Cu") (net 2))
