File: electronics_design/SmartLampSE.kicad_pcb (KiCad board)
At the start: 2 copper layers, 60 x 60 mm, 14 parts, among them J1 Screw_Terminal_01x02, M1 PIC16F886-IP, U1 L7805, Y1 Crystal

Commit message: Fix some widths
Other:
- board outline removed
Changed lines of the file:
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@@
     (pad_to_mask_clearance 0)
     (pcbplotparams
-      (layerselection 0x00010fc_ffffffff)
+      (layerselection 0x0000000_fffffffe)
       (plot_on_all_layers_selection 0x0000000_00000000)
       (disableapertmacros false)
@@
       (sketchpadsonfab false)
       (subtractmaskfromsilk false)
-      (outputformat 1)
+      (outputformat 2)
       (mirror false)
-      (drillshape 1)
+      (drillshape 2)
       (scaleselection 1)
       (outputdirectory "")
@@
     )
   )
-  (gr_circle (center 166 79) (end 166 83)
-    (stroke (width 0.2) (type solid)) (fill none) (layer "B.Cu"))
+  (gr_circle (center 166 79) (end 170 79)
+    (stroke (width 0.3) (type solid)) (fill none) (layer "B.Cu"))
+  (gr_circle (center 166 79) (end 168 79)
+    (stroke (width 0.3) (type solid)) (fill none) (layer "B.Cu"))
+  (gr_circle (center 116 129) (end 118 129)
+    (stroke (width 0.3) (type solid)) (fill none) (layer "B.Cu"))
   (gr_rect (start 91 54) (end 191 154)
-    (stroke (width 0.2) (type solid)) (fill none) (layer "B.Cu"))
-  (gr_circle (center 116 79) (end 116 83)
-    (stroke (width 0.2) (type solid)) (fill none) (layer "B.Cu"))
-  (gr_circle (center 116 129) (end 116 133)
-    (stroke (width 0.2) (type solid)) (fill none) (layer "B.Cu"))
-  (gr_circle (center 166 129) (end 166 133)
-    (stroke (width 0.2) (type solid)) (fill none) (layer "B.Cu"))
+    (stroke (width 0.6) (type solid)) (fill none) (layer "B.Cu"))
+  (gr_circle (center 116 79) (end 120 79)
+    (stroke (width 0.3) (type solid)) (fill none) (layer "B.Cu"))
+  (gr_circle (center 116 129) (end 120 129)
+    (stroke (width 0.3) (type solid)) (fill none) (layer "B.Cu"))
+  (gr_circle (center 116 79) (end 118 79)
+    (stroke (width 0.3) (type solid)) (fill none) (layer "B.Cu"))
+  (gr_circle (center 166 129) (end 168 129)
+    (stroke (width 0.3) (type solid)) (fill none) (layer "B.Cu"))
+  (gr_rect (start 111 74) (end 171 134)
+    (stroke (width 0.6) (type solid)) (fill none) (layer "B.Cu"))
+  (gr_circle (center 166 129) (end 170 129)
+    (stroke (width 0.3) (type solid)) (fill none) (layer "B.Cu"))
   (gr_rect (start 121 75) (end 161 85)
     (stroke (width 0.2) (type default)) (fill none) (layer "F.SilkS"))
-  (gr_circle (center 166 79) (end 168 79)
-    (stroke (width 0.2) (type solid)) (fill none) (layer "Edge.Cuts"))
-  (gr_circle (center 116 129) (end 118 129)
-    (stroke (width 0.2) (type solid)) (fill none) (layer "Edge.Cuts"))
-  (gr_circle (center 116 79) (end 118 79)
-    (stroke (width 0.2) (type solid)) (fill none) (layer "Edge.Cuts"))
-  (gr_circle (center 166 129) (end 168 129)
-    (stroke (width 0.2) (type solid)) (fill none) (layer "Edge.Cuts"))
-  (gr_rect (start 111 74) (end 171 134)
-    (stroke (width 0.2) (type solid)) (fill none) (layer "Edge.Cuts"))
   (gr_text "+" (at 119.84 122.52) (layer "B.Cu")
     (effects (font (size 4 4) (thickness 1) bold) (justify left bottom mirror))
   )
   (gr_text "GND(B)" (at 164.49 112.61) (layer "B.Cu")
-    (effects (font (size 1.2 1.2) (thickness 0.25) bold) (justify left bottom mirror))
+    (effects (font (size 1.2 1.2) (thickness 0.3) bold) (justify left bottom mirror))
   )
   (gr_text "AN12\n" (at 162.83 106.48) (layer "B.Cu")
-    (effects (font (size 1.2 1.2) (thickness 0.25) bold) (justify left bottom mirror))
+    (effects (font (size 1.2 1.2) (thickness 0.3) bold) (justify left bottom mirror))
   )
   (gr_text "SPI" (at 153.03 84.62 90) (layer "B.Cu")
-    (effects (font (size 1.4 1.4) (thickness 0.3) bold) (justify left bottom mirror))
+    (effects (font (size 1.5 1.5) (thickness 0.3) bold) (justify left bottom mirror))
   )
   (gr_text "I2C\n" (at 153.21 120 90) (layer "B.Cu")
-    (effects (font (size 1.4 1.4) (thickness 0.3) bold) (justify left bottom mirror))
+    (effects (font (size 1.5 1.5) (thickness 0.3) bold) (justify left bottom mirror))
   )
   (gr_text "SDO\n" (at 157.95 86.32) (layer "B.Cu")
@@
   )
   (gr_text "CCMP1" (at 164.31 99) (layer "B.Cu")
-    (effects (font (size 1.2 1.2) (thickness 0.25) bold) (justify left bottom mirror))
+    (effects (font (size 1.2 1.2) (thickness 0.3) bold) (justify left bottom mirror))
   )
   (gr_text "SDA" (at 157.87 121.6) (layer "B.Cu")
@@
   )
   (gr_text "RX(O)" (at 163.27 115.15) (layer "B.Cu")
-    (effects (font (size 1.2 1.2) (thickness 0.25) bold) (justify left bottom mirror))
+    (effects (font (size 1.2 1.2) (thickness 0.3) bold) (justify left bottom mirror))
   )
   (gr_text "TX(Y)" (at 162.75 117.7) (layer "B.Cu")
-    (effects (font (size 1.2 1.2) (thickness 0.25) bold) (justify left bottom mirror))
+    (effects (font (size 1.2 1.2) (thickness 0.3) bold) (justify left bottom mirror))
   )
   (gr_text "UART" (at 153 109 90) (layer "B.Cu")
@@
   )
   (gr_text "IO" (at 153 97 90) (layer "B.Cu")
-    (effects (font (size 1.4 1.4) (thickness 0.3) bold) (justify left bottom mirror))
+    (effects (font (size 1.5 1.5) (thickness 0.3) bold) (justify left bottom mirror))
   )
   (gr_text "↓" (at 132.26 80.54 145) (layer "B.Cu")
@@
   )
   (gr_text "AN10\n" (at 162.86 103.78) (layer "B.Cu")
-    (effects (font (size 1.2 1.2) (thickness 0.25) bold) (justify left bottom mirror))
+    (effects (font (size 1.2 1.2) (thickness 0.3) bold) (justify left bottom mirror))
   )
   (gr_text "AN08\n" (at 162.87 101.32) (layer "B.Cu")
-    (effects (font (size 1.2 1.2) (thickness 0.25) bold) (justify left bottom mirror))
+    (effects (font (size 1.2 1.2) (thickness 0.3) bold) (justify left bottom mirror))
   )
   (gr_text "RB5" (at 161.91 89.3) (layer "B.Cu")
@@
   )
   (gr_text "RB4" (at 161.83 91.73) (layer "B.Cu")
-    (effects (font (size 1.2 1.2) (thickness 0.25) bold) (justify left bottom mirror))
-  )
-  (gr_text "TRIANGLE POINTS\nTO PIN1" (at 159.76 79.34) (layer "B.Cu")
     (effects (font (size 1.2 1.2) (thickness 0.3) bold) (justify left bottom mirror))
   )
+  (gr_text "TRIANGLE POINTS\nTO PIN1" (at 160.7 79.75) (layer "B.Cu")
+    (effects (font (size 1.5 1.5) (thickness 0.3) bold) (justify left bottom mirror))
+  )
   (gr_text "-" (at 119.08 103.02 90) (layer "B.Cu")
